Commit message: Add endurance test script and update sensor configurations
- Introduced `endurance_test.py` for autonomous loop navigation and logging during endurance testing.
- Added new STL files for models: `Model_v2.stl` and `RPLiDAR_s2.stl`.
- Modified `jetson_sensor_bridge.py` to update sensor indexing and adjust serial port settings.
- Enhanced `ultrasonic_fusion_node.py` with hard stop functionality and improved sensor handling.
- Updated `wheel_odom_node.py` to change the default serial port.
- Adjusted URDF for the robot to correct the orientation of the laser frame and ultrasonic sensors.

File: urdf/mobile_robot_v2.urdf.xacro (robot description, xacro)
@@ -166,9 +166,9 @@
         <parent link="chassis"/>
         <child link="laser_frame"/>
-        <origin xyz="0.257 0 0.075" rpy="0 0 0"/>
+        <origin xyz="0.257 0 0.075" rpy="0 0 3.14159"/>
     </joint>
     <link name="laser_frame">
         <visual>
-            <origin xyz="0 0 0" rpy="0 0 0"/>
+            <origin xyz="0 0 0" rpy="0 0 3.14159"/>
             <geometry>
                 <!-- <cylinder length="0.04" radius="0.038"/> -->
@@ -178,8 +178,8 @@
         </visual>
         <collision>
-            <origin xyz="0 0 0" rpy="0 0 0"/>
-            <geometry>
-                <!-- <cylinder length="0.04" radius="0.038"/> -->
-                <mesh filename="package://mobile_robot/meshes/RPLiDAR_s2.stl" scale="0.001 0.001 0.001"/>
+            <origin xyz="0 0 0" rpy="0 0 3.14159"/>
+            <geometry>
+                <cylinder length="0.04" radius="0.038"/>
+                <!-- <mesh filename="package://mobile_robot/meshes/RPLiDAR_s2.stl" scale="0.001 0.001 0.001"/> -->
             </geometry>
         </collision>
@@ -222,10 +222,10 @@
         </link>
     </xacro:macro>
-    <joint name="us_top_left_joint" type="fixed">
+    <!-- <joint name="us_top_left_joint" type="fixed">
         <parent link="chassis"/>
         <child link="us_top_left_link"/>
         <origin xyz="0.35 0.17 0.48" rpy="0 0 0"/>
     </joint>
-    <xacro:ultrasonic_link name="us_top_left"/>
+    <xacro:ultrasonic_link name="us_top_left"/> -->
     <joint name="us_top_right_joint" type="fixed">
         <parent link="chassis"/>
